File: Diff_probe.kicad_pcb (KiCad board)
At the start: 4 copper layers, 61.5 x 45 mm, 82 parts, among them J1 Conn_01x03_Male, J2 TYPE-C-31-M-12, J3 Conn_01x03_Male, J4 Conn_01x03_Male, J5 Conn_01x03_Male, U1 OPA2356xxD, U2 OPA2356xxD, U3 XC6206PxxxMR

Commit message: As ordered prototype 20230121
Parts:
- added JP9: Jumper_3_Open, Jumper:SolderJumper-3_P2.0mm_Open_TrianglePad1.0x1.5mm, F.Cu at (158.4, 30.2)
- added R41: R_100, Resistor_SMD:R_0805_2012Metric, F.Cu at (151.8, 24.3)
- added R42: R_100, Resistor_SMD:R_0805_2012Metric, F.Cu at (151.8, 26.3)
- C1, C3, C4: value C_Polarized_Small -> C_10uF_Tant
- C10, C11, C6, C9: value C_Small -> C_47pF
- C2, C5, C7, C8: value C_Small -> C_100nF
- R10, R19, R37, R38: value R_Small -> R_47
- R11, R20, R39, R40: value R_Small -> R_DNP
- R15, R17, R29, R31, R33, R34, R6, R7: value R_Small -> R_10k
- R16, R18, R30, R32, R35, R36, R8, R9: value R_Small -> R_40k
- moved C3 1.96 mm to (151.2, 30.6)
- moved U3 1.96 mm to (154.2, 31.1)
Connections:
- J1 pad 3: unconnected-(J1-Pad3) -> +5V
- J3 pad 3: unconnected-(J3-Pad3) -> +5V
- J4 pad 3: unconnected-(J4-Pad3) -> +5V
- J5 pad 3: unconnected-(J5-Pad3) -> +5V
- U3 pad 2: +2V5 -> Net-(U3-Pad2)
Routing:
- net Net-(R41-Pad2): track 0.00 -> 8.16 mm
- net +2V5: track 17.1 -> 20.5 mm
- net Net-(U3-Pad2): track 0.00 -> 3.30 mm
- net +5V: track 8.32 -> 8.97 mm, vias 5 -> 6
- net GND: track 58.0 -> 57.8 mm, vias 10 -> 11
Other:
- board text added: "2.5V MID"
- board text added: "USE: 5V can be powered from 5V or 3V3 depending on the microcontroller used. Do NOT connect USB and 3V3 at the same time. USB intended for using this as a scope probe. SAFETY: Do NOT bridge the 2512 1MOhm resistors. Do NOT put a capacitor between board LV and ground; ground LV side properly. Use UL rated 1MOhm resistors if using HV (e.g. 400V) and be careful, HV is dangerous."
