File: Diff_probe.kicad_sch (KiCad schematic)
At the start: 82 parts

Commit message: As ordered prototype 20230121
Parts:
- added JP9: (no value), symbol Jumper:Jumper_3_Open
- added R41, R42: (no value), symbol Device:R_Small
Connections:
- net +2V5: now also JP9.2 (C); no longer U3.2 (VO)
- net +5V: now also J1.3 (Pin_3), J3.3 (Pin_3), J4.3 (Pin_3), J5.3 (Pin_3), R41.1
- net GND: now also R42.2
- new net: JP9.3 (B), R41.2, R42.1
- new net: JP9.1 (A), U3.2 (VO)
Other:
- moved on the sheet: C1, C2, C3, C4, C5, C7, C8, U3
